File: EBB/EBB.kicad_pcb (KiCad board)
At the start: 2 copper layers, 9 parts, among them J3 Motor_Driver, J6 Motor

Commit message: Added some body about the blocker design and a table with the bill of materials. Not currently building.
Parts:
- added G***: LOGO, LOGO, F.Cu at (196.8, 102.9)
- moved C1 31.9 mm to (189.9, 78.0), turned to 90 degrees
- renumbered J3 to Driver
Connections:
- Pico1 pad 10: (no net) -> GND
- Pico1 pad 11: (no net) -> GND
- Pico1 pad 15: (no net) -> GND
- Pico1 pad 16: (no net) -> GND
- Pico1 pad 17: (no net) -> GND
- Pico1 pad 4: (no net) -> GND
- Pico1 pad 5: (no net) -> GND
- Pico1 pad 6: (no net) -> GND
- Pico1 pad 7: (no net) -> GND
- Pico1 pad 9: (no net) -> GND
Routing:
- net +5V: track 95.5 -> 93.9 mm
- net GND: vias 0 -> 9
- added copper zone on B.Cu, net GND
Other:
- board outline added: 21.6 x 70.5 mm
- board text added: "Stephen Hofmann Derek Jenkins Thomas Stay Andrew Koebbe"
- board text added: "VSYS"
